Commit message: Correções e Atualização README

File: urdf/oakd.urdf.xacro (robot description, xacro)
@@ -24,5 +24,5 @@
                 <geometry>
                     <mesh
-                        filename="package://gazebo_project/meshes/${name}_${model}.dae"
+                        filename="package://trekking_2025/meshes/${name}_${model}.dae"
                         scale="1 1 1" />
                 </geometry>

File: urdf/smart_autonomous_car.urdf (robot description, URDF)
Before this commit: robot robot, 8 links, 7 joints
Links:
- link link_chassis: geometry collision box size=2.4 1.0 1.0; visual mesh filename=package://trekking_2025/meshes/Chassi_RC.obj scale=0.15 0.14 0.156

File: urdf/tutorial_robot.urdf (robot description, URDF)
Before this commit: robot robot, 8 links, 7 joints
Links:
- link link_chassis: geometry collision box size=2.4 1.0 1.0; visual mesh filename=package://trekking_2025/meshes/Chassi_RC.obj scale=0.012 0.012 0.013
