Commit message: Escala do Robô e Simulação no RVIZ2 corrigidas

File: urdf/robot.urdf (robot description, URDF)
Before this commit: robot robot, 1 links, 0 joints
Links:
- added link front_left_wheel; collision sphere radius=0.06; visual cylinder length=0.07 radius=0.06
- added link front_left_wheel_steering_link
- added link front_right_wheel; collision sphere radius=0.06; visual cylinder length=0.07 radius=0.06
- added link front_right_wheel_steering_link
- added link link_chassis; collision box size=0.5 0.35 0.22; visual mesh filename=package://trekking_2025/meshes/Chassi_RC.obj scale=0.042 0.042 0.042
- added link rear_left_wheel; collision sphere radius=0.06; visual cylinder length=0.07 radius=0.06
- added link rear_right_wheel; collision sphere radius=0.06; visual cylinder length=0.07 radius=0.06
Joints:
- added joint front_left_wheel_rotating_joint: type revolute, parent front_left_wheel_steering_link, child front_left_wheel, origin xyz=0 0 0 rpy=0 0 0, axis 0 0 1, limit lower=-1.79769e+308 upper=1.79769e+308 effort=100000 velocity=1000
- added joint front_left_wheel_steering_joint: type revolute, parent link_chassis, child front_left_wheel_steering_link, origin xyz=0.25 0.175 0.06 rpy=-1.56 0 0, axis 0 -1 0, limit lower=-0.8727 upper=0.8727 effort=100000 velocity=1000
- added joint front_right_wheel_rotating_joint: type revolute, parent front_right_wheel_steering_link, child front_right_wheel, origin xyz=0 0 0 rpy=0 0 0, axis 0 0 1, limit lower=-1.79769e+308 upper=1.79769e+308 effort=100000 velocity=1000
- added joint front_right_wheel_steering_joint: type revolute, parent link_chassis, child front_right_wheel_steering_link, origin xyz=0.25 -0.175 0.06 rpy=-1.56 0 0, axis 0 -1 0, limit lower=-0.8727 upper=0.8727 effort=100000 velocity=1000
- added joint joint_base_link_chassis: type fixed, parent base_link, child link_chassis, origin xyz=0 0 0 rpy=0 0 0
- added joint rear_left_wheel_joint: type revolute, parent link_chassis, child rear_left_wheel, origin xyz=-0.25 0.175 0.06 rpy=1.56 0 0, axis 0 0 1, limit lower=-1.79769e+308 upper=1.79769e+308 effort=100000 velocity=1000
- added joint rear_right_wheel_joint: type revolute, parent link_chassis, child rear_right_wheel, origin xyz=-0.25 -0.175 0.06 rpy=1.56 0 0, axis 0 0 1, limit lower=-1.79769e+308 upper=1.79769e+308 effort=100000 velocity=1000

File: urdf/smart_autonomous_car.urdf (robot description, URDF)
Before this commit: robot robot, 8 links, 7 joints
Links:
- link link_chassis: geometry collision box size=2.4 1.0 1.0; visual mesh filename=package://gazebo_project/meshes/smart_car.obj scale=0.012 0.012 0.013
