Commit message: Lidar 50%

File: urdf/hokuyo_ust10lx.urdf.xacro (robot description, xacro)
@@ -3,4 +3,5 @@
   <xacro:include filename="$(find trekking_2025)/urdf/materials.urdf.xacro"/>
   <xacro:macro name="sensor_hokuyo_ust10lx" params="name visualize:=false parent *origin color min_angle:=-2.3562 max_angle:=2.3562">
+    <!-- Fixed joint to parent -->
     <joint name="${name}_joint" type="fixed">
       <xacro:insert_block name="origin" />
@@ -8,4 +9,5 @@
       <child link="${name}_link"/>
     </joint>
+    <!-- Sensor body -->
     <link name="${name}_link">
       <collision>
@@ -28,14 +30,10 @@
       </inertial>
     </link>
-    <!-- Hokuyo sensor for simulation -->
-    <sensor_hokuyo_ust_gazebo name="${name}" visualize="${visualize}" min_angle="${min_angle}" max_angle="${max_angle}"/>
-    <xacro:color_gazebo parent="${name}_link" color="${color}"/>
-  </xacro:macro>
-  <xacro:macro name="sensor_hokuyo_ust_gazebo" params="name visualize min_angle max_angle">
+    <!-- Sensor configuration for Ignition -->
     <gazebo reference="${name}_link">
       <sensor name="${name}_sensor" type="gpu_lidar">
         <pose>0 0 0 0 0 0</pose>
         <topic>${name}/scan</topic>
-        <update_rate>40</update_rate>
+        <update_rate>10</update_rate>
         <ray>
           <scan>
@@ -48,5 +46,5 @@
             <vertical>
               <samples>1</samples>
-              <resolution>1</resolution>
+              <resolution>0.01</resolution>
               <min_angle>0</min_angle>
               <max_angle>0</max_angle>
@@ -58,15 +56,10 @@
             <resolution>0.01</resolution>
           </range>
-          <!--noise>
-            <type>gaussian</type>
-            <mean>0.0</mean>
-            <stddev>0.01</stddev>
-          </noise-->
         </ray>
         <always_on>1</always_on>
-        <!--visualize>${visualize}</visualize-->
-        <visualize>true</visualize>
+        <visualize>${visualize}</visualize>
       </sensor>
     </gazebo>
+    <xacro:color_gazebo parent="${name}_link" color="${color}"/>
   </xacro:macro>
 </robot>
